Commit message: retrofit to controller packages to fit cobot joint config

File: cobot_description/description/new_mycobot_pro_320_pi_2022.urdf (robot description, URDF)
Before this commit: robot firefighter, 7 links, 6 joints
Links:
- link base: geometry collision mesh filename=package://cobot_description/assets/base.dae; visual mesh filename=package://cobot_description/assets/base.dae
- link link1: geometry collision mesh filename=package://cobot_description/assets/link1.dae; visual mesh filename=package://cobot_description/assets/link1.dae
- link link2: geometry collision mesh filename=package://cobot_description/assets/link2.dae; visual mesh filename=package://cobot_description/assets/link2.dae
- link link3: geometry collision mesh filename=package://cobot_description/assets/link3.dae; visual mesh filename=package://cobot_description/assets/link3.dae
- link link4: geometry collision mesh filename=package://cobot_description/assets/link4.dae; visual mesh filename=package://cobot_description/assets/link4.dae
- link link5: geometry collision mesh filename=package://cobot_description/assets/link5.dae; visual mesh filename=package://cobot_description/assets/link5.dae
- link link6: geometry collision mesh filename=package://cobot_description/assets/link6.dae; visual mesh filename=package://cobot_description/assets/link6.dae
Joints:
- removed joint joint2_to_joint1
- removed joint joint3_to_joint2
- removed joint joint4_to_joint3
- removed joint joint5_to_joint4
- removed joint joint6_to_joint5
- removed joint joint6output_to_joint6
- added joint j1: type revolute, parent base, child link1, origin xyz=0 0 0.1739 rpy=0 0 0, axis 0 0 1, limit lower=-2.93 upper=2.93 effort=1000.0 velocity=1.0
- added joint j2: type revolute, parent link1, child link2, origin xyz=0 -0.08878 0 rpy=0 -1.5708 1.5708, axis 0 0 1, limit lower=-2.35 upper=2.35 effort=1000.0 velocity=1.0
- added joint j3: type revolute, parent link2, child link3, origin xyz=0.135 0 -0.08878 rpy=0 0 0, axis 0 0 1, limit lower=-2.53 upper=2.53 effort=1000.0 velocity=1.0
- added joint j4: type revolute, parent link3, child link4, origin xyz=0.120 0 0.08878 rpy=0 0 1.57080, axis 0 0 1, limit lower=-2.53 upper=2.53 effort=1000.0 velocity=1.0
- added joint j5: type revolute, parent link4, child link5, origin xyz=0 -0.095 0 rpy=1.5708 0 0, axis 0 0 1, limit lower=-2.93 upper=2.93 effort=1000.0 velocity=1.0
- added joint j6: type revolute, parent link5, child link6, origin xyz=0 0.0655 0 rpy=-1.5708 0 0, axis 0 0 1, limit lower=-3.14 upper=3.14 effort=1000.0 velocity=1.0

Commit message: used new urdf for moveit2 setup, changed damping and psring settings to 100 within nvidia isaac launch file now explicitely loads in ros2 control nodes TODO create a jogger script to send position commands to moveit, and have trajectories replay within isaacsim

File: cobot_description/description/new_mycobot_pro_320_pi_2022.urdf (robot description, URDF)
Before this commit: robot firefighter, 7 links, 6 joints
Joints:
- removed joint j1
- removed joint j2
- removed joint j3
- removed joint j4
- removed joint j5
- removed joint j6
- added joint joint2_to_joint1: type revolute, parent base, child link1, origin xyz=0 0 0.1739 rpy=0 0 0, axis 0 0 1, limit lower=-2.93 upper=2.93 effort=1000.0 velocity=1.0
- added joint joint3_to_joint2: type revolute, parent link1, child link2, origin xyz=0 -0.08878 0 rpy=0 -1.5708 1.5708, axis 0 0 1, limit lower=-2.35 upper=2.35 effort=1000.0 velocity=1.0
- added joint joint4_to_joint3: type revolute, parent link2, child link3, origin xyz=0.135 0 -0.08878 rpy=0 0 0, axis 0 0 1, limit lower=-2.53 upper=2.53 effort=1000.0 velocity=1.0
- added joint joint5_to_joint4: type revolute, parent link3, child link4, origin xyz=0.120 0 0.08878 rpy=0 0 1.57080, axis 0 0 1, limit lower=-2.53 upper=2.53 effort=1000.0 velocity=1.0
- added joint joint6_to_joint5: type revolute, parent link4, child link5, origin xyz=0 -0.095 0 rpy=1.5708 0 0, axis 0 0 1, limit lower=-2.93 upper=2.93 effort=1000.0 velocity=1.0
- added joint joint6output_to_joint6: type revolute, parent link5, child link6, origin xyz=0 0.0655 0 rpy=-1.5708 0 0, axis 0 0 1, limit lower=-3.14 upper=3.14 effort=1000.0 velocity=1.0
