Commit message: added simple RL environment training

File: cobot_description/description/robot.urdf (robot description, URDF)
Before this commit: robot cobot_description, 7 links, 6 joints
Links:
- removed link link_1
- added link w_j6末端, mass 1e-09; collision mesh filename=package://cobot_description/assets/bottom.stl; collision mesh filename=package://cobot_description/assets/c3_assy.stl
- link ground_link: geometry collision mesh filename=package://cobot_description/assets/link_1.stl; collision mesh filename=package://cobot_description/assets/w_pi模组.stl
- link link_6: geometry collision mesh filename=package://cobot_description/assets/w_j6部分.stl; collision mesh filename=package://cobot_description/assets/w_j6部分__2.stl
Joints:
- joint joint2_to_joint1: child link_1 -> link_2; limit effort=10 velocity=10 -> lower=-3.141592653589793 upper=3.141592653589793 effort=10 velocity=10; origin xyz=-4.83452e-05 -0.0425776 0.0466572 rpy=-1.5708 -0 -3.14159 -> xyz=-4.83452e-05 -0.00581885 0.0964 rpy=0 0 3.14159; type fixed -> revolute
- joint joint3_to_joint2: child link_2 -> link_3; origin xyz=0 -0.0497428 -0.0367587 rpy=1.5708 0 0 -> xyz=-0.0479996 0.000184098 0.0784 rpy=-1.5708 0 1.56696; parent link_1 -> link_2
- joint joint4_to_joint3: child link_3 -> link_4; origin xyz=-0 -0.0629 0.0784 rpy=-1.5708 0.258432 3.14159 -> xyz=0 -0.134451 -0.00841215 rpy=0 0 -3.1366; parent link_2 -> link_3
- joint joint5_to_joint4: child link_4 -> link_5; origin xyz=0 -0.134451 -0.00841215 rpy=-0 0 -2.92416 -> xyz=0 0.12 -0.0019 rpy=-3.14159 0 3.12542; parent link_3 -> link_4
- joint joint6_to_joint5: child link_5 -> link_6; origin xyz=0 0.12 -0.0019 rpy=-3.14159 -0 -2.55731 -> xyz=5.5683e-08 0.045 -0.0495147 rpy=-1.5708 -0.0123971 3.14159; parent link_4 -> link_5
- joint joint6output_to_joint6: child link_6 -> w_j6末端; origin xyz=5.5683e-08 0.045 -0.0495147 rpy=-1.5708 -0 -3.14159 -> xyz=0 0.045 -0.0497 rpy=-1.5708 0.00892376 -3.14159; parent link_5 -> link_6
