Commit message: added frame towards end effector tip added ballpark estimate mass and interias for each major link converted to usda format readably by isaaclab 5.1 using isaacsim5.1 save as method USE THE ROBOT FOLDER WITH NO NUMBER SUFFIX, BEST WORKING VERSION

File: cobot_description/robot.urdf (robot description, URDF)
Before this commit: robot cobot_description, 7 links, 6 joints
Links:
- added link ultrasound_tip, mass 1e-9
- link ground_link: mass 1.200 -> 1.1; geometry collision mesh filename=package://cobot_description/assets/link_1.stl; collision mesh filename=package://cobot_description/assets/w_pi模组.stl
- link link_2: mass 0.650 -> 0.65; geometry collision mesh filename=package://cobot_description/assets/link_2.stl; visual mesh filename=package://cobot_description/assets/link_2.stl
- link link_3: mass 0.550 -> 0.55; geometry collision mesh filename=package://cobot_description/assets/w_j3部分.stl; collision mesh filename=package://cobot_description/assets/w_j3部分__2.stl
- link link_4: mass 0.400 -> 0.4; geometry collision mesh filename=package://cobot_description/assets/w_j4部分.stl; collision mesh filename=package://cobot_description/assets/w_j4部分__2.stl
- link link_5: mass 0.300 -> 0.35; geometry collision mesh filename=package://cobot_description/assets/link_5.stl; visual mesh filename=package://cobot_description/assets/link_5.stl
- link link_6: mass 0.120 -> 0.31; geometry collision mesh filename=package://cobot_description/assets/w_j6部分.stl; collision mesh filename=package://cobot_description/assets/w_j6部分__2.stl
- link w_j6: mass 0.080 -> .307; geometry collision mesh filename=package://cobot_description/assets/bottom.stl; collision mesh filename=package://cobot_description/assets/c3_assy.stl
Joints:
- added joint ultrasound_tip_frame: type fixed, parent w_j6, child ultrasound_tip, origin xyz=-0.0732943 3.33067e-16 -0.0586367 rpy=1.52382 -7.37084e-15 -1.5708, axis 0 0 0
- joint joint2_to_joint1: limit lower=-2.87979 upper=2.87979 effort=3.0 velocity=3.0 -> lower=-2.93125 upper=2.93125 effort=5 velocity=2.8
- joint joint3_to_joint2: limit lower=-2.87979 upper=2.87979 effort=2.5 velocity=3.0 -> lower=-2.35619 upper=2.35619 effort=5 velocity=2.8
- joint joint4_to_joint3: limit lower=-2.87979 upper=2.87979 effort=2.0 velocity=3.0 -> lower=-2.53073 upper=2.53073 effort=4 velocity=2.8
- joint joint5_to_joint4: limit lower=-2.87979 upper=2.87979 effort=1.5 velocity=3.0 -> lower=-2.53073 upper=2.53073 effort=2 velocity=3.2
- joint joint6_to_joint5: limit lower=-2.87979 upper=2.87979 effort=1.0 velocity=3.0 -> lower=-2.93215 upper=2.93215 effort=2 velocity=3.2
- joint joint6output_to_joint6: limit lower=-3.05433 upper=3.05433 effort=0.8 velocity=3.0 -> lower=-3.141592653589793 upper=3.141592653589793 effort=1.5 velocity=3.5
